File: USB-UART.kicad_pcb (KiCad board)
At the start: 2 copper layers, 39 x 19 mm, 19 parts, among them J1 Connector, USB-TYPE-C-16P, J2 Conn_01x09_Pin, J3 Conn_01x06, J4 Conn_01x09_Pin, U1 FT232RL

Commit message: add: github link
Other:
- board text added: "https://github.com/wirenux/USBC-UART"
Changed lines of the file:
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@@
+		)
+	)
+	(gr_text "https://github.com/wirenux/USBC-UART"
+		(at 135 95 0)
+		(layer "B.SilkS")
+		(effects
+			(font
+				(size 0.5 0.5)
+				(thickness 0.125)
+				(bold yes)
+			)
+			(justify left bottom mirror)
 		)
 	)
